File: kicad/hood-control.kicad_pcb (KiCad board)
At the start: 2 copper layers, 80 x 55 mm, 40 parts, among them J1 Hoodcontrol, J2 FTDI Serial Flash, J3 Frontpanel, J4 Reset, J5 Flash/Run, J6 PWR_IN, SW1 Reset, SW2 Flash, U1 ESP-12E, U2 4050, U3 74HCT08, U4 Stepdown 3.3V

Commit message: Platzierung fertig, vor dem Routen
Parts:
- U4: footprint Connector_PinHeader_2.54mm:PinHeader_1x03_P2.54mm_Vertical -> hood-control:TPS63802_Module_25.8x13.0mm
- moved C1 15.8 mm to (42.7, 52.4), turned to -90 degrees
- moved C6 15.2 mm to (63.3, 65.5)
- moved TP2 9.34 mm to (37.9, 65.3)
- moved TP4 9.23 mm to (41.1, 65.3)
- moved J5 8.79 mm to (27.1, 65.2)
- moved U4 4.21 mm to (54.6, 54.1), turned to -90 degrees
- moved TP1 3.43 mm to (69.1, 52.7), turned to -90 degrees
- moved C8 2.43 mm to (59.7, 35.0)
- moved TP3 2.05 mm to (69.1, 55.8), turned to -90 degrees
- moved C3 1.32 mm to (42.0, 48.2)
- moved SW2 0.93 mm to (36.0, 54.2)
Connections:
- U4 pad 1: unconnected-(U4-IN-Pad1) -> /5V_IN
Other:
- board text added: "or/w or gn/w bl bl/w gn br/w br"
- board text removed: "U4 TPS63802-Modul 26 x 12,5 mm Footprint erst nach Vermessung"
- board text removed: "orwe or gnwe bl blwe gn brwe br"
