File: kicad/hood-control.kicad_pcb (KiCad board)
At the start: 2 copper layers, 80 x 55 mm, 40 parts, among them J1 Hoodcontrol, J2 FTDI Serial Flash, J3 Frontpanel, J4 Reset, J5 Flash/Run, J6 PWR_IN, SW1 Reset, SW2 Flash, U1 ESP-12E, U2 4050, U3 74HCT08, U4 Stepdown 3.3V

Commit message: Route the board and add fabrication outputs
The PCB is fully routed: 174 track segments and 6 vias on two layers, with a
filled GND plane on B.Cu (3531 mm², one contiguous polygon). Every ground
connection hangs on that plane except U1's SMD pad 15, which reaches it
through two redundant vias.

Signals stay on F.Cu wherever they can (133 of 174 segments) so the back side
remains a solid reference; only unavoidable crossings dip to B.Cu.

Power nets get their own netclass: 0.6 mm tracks and 0.8/0.4 mm vias, signals
stay at 0.25 mm. The tightest copper clearance is 0.200 mm and the smallest
drill 0.30 mm — inside PCBWay's 6/6 mil class, but 8/8 mil would no longer
fit, so the order has to specify 6/6.

kicad/fab/ holds the seven Gerber layers, the PTH/NPTH Excellon files, the job
file and a ready-to-upload zip, plus FAB.md with the order parameters.

DRC: 0 violations, 0 unconnected items. The four keepout hits and the nine
schematic-parity hints are the documented, intentional ones.

Co-Authored-By: Claude Opus 5 <noreply@anthropic.com>
Routing:
- net VCC: track 0.00 -> 125.1 mm
- net /SCAN: track 0.00 -> 60.1 mm
- net /GPIO12: track 0.00 -> 59.2 mm
- net /5V_IN: track 0.00 -> 57.2 mm
- net /GPIO14: track 0.00 -> 53.6 mm
- net /RST: track 0.00 -> 52.2 mm
- net /GPIO13: track 0.00 -> 47.7 mm, vias 0 -> 1
- net /LED_CH_1: track 0.00 -> 38.9 mm
- net /GPIO0: track 0.00 -> 38.8 mm
- net /LED_CH_2: track 0.00 -> 31.3 mm
- net /BTN_CH_1: track 0.00 -> 29.4 mm
- net /GPIO5: track 0.00 -> 29.2 mm
- net /BTN_CH_2: track 0.00 -> 26.9 mm
- net /GPIO4: track 0.00 -> 23.7 mm, vias 0 -> 1
- net /ESP_RXD: track 0.00 -> 20.1 mm, vias 0 -> 1
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- added copper zone on B.Cu, net GND
Other:
- board text added: "WayWayWay"

Commit message: Rev 0.3: decouple U3 from the hood's key matrix, fix channel mapping
Bring-up of the rev 0.2 boards showed that U3's push-pull outputs on the
key lines cause boot loops and phantom key presses. D3/D4 now sit in
series behind U3 (the board can only pull a line high, never hold it
low) and R7/R8 keep U3's inputs low until the firmware runs.

Firmware drives GPIO12/14 actively (LOW = release, HIGH = press) from
the very start of setup(), and swaps the LED and button pins, which
arrive the other way round than the perfboard firmware assumed.

DESIGN.md documents the findings and corrects the old assumption that
D1/D2 protected the key lines.

Co-Authored-By: Claude Opus 5.5 <noreply@anthropic.com>
Parts:
- added D3: 1N4148, Diode_THT:D_DO-35_SOD27_P2.54mm_Vertical_AnodeUp, F.Cu at (83.4, 52.7)
- added D4: 1N4148, Diode_THT:D_DO-35_SOD27_P2.54mm_Vertical_AnodeUp, F.Cu at (74.2, 52.7)
- added R7: 10k, Resistor_THT:R_Axial_DIN0207_L6.3mm_D2.5mm_P2.54mm_Vertical, F.Cu at (87.9, 52.7)
- added R8: 10k, Resistor_THT:R_Axial_DIN0207_L6.3mm_D2.5mm_P2.54mm_Vertical, F.Cu at (78.8, 52.7)
- TP4: value 3V3 -> 3.3V
- moved R5 30.4 mm to (71.8, 29.2), turned to 90 degrees
Connections:
- U3 pad 3: /BTN_CH_1 -> Net-(D3-A)
- U3 pad 6: /BTN_CH_2 -> Net-(D4-A)
Routing:
- net /SCAN: track 60.1 -> 43.4 mm
- net /BTN_CH_1: track 29.4 -> 21.0 mm
- net /GPIO14: track 53.6 -> 61.4 mm, vias 0 -> 2
- net /GPIO12: track 59.2 -> 66.6 mm, vias 0 -> 2
- net /BTN_CH_2: track 26.9 -> 32.0 mm
- net Net-(D4-A): track 0.00 -> 3.14 mm
- net Net-(D3-A): track 0.00 -> 2.93 mm
Other:
- board text added: "ESP Haubensteuerung für Gutmann Sombra v0.3"
- board text removed: "ESP Haubensteuerung für Gutmann Sombra v0.2"
