File: kicad/hood-control.kicad_sch (KiCad schematic)
At the start: 32 parts, among them J1 Hoodcontrol, J2 FTDI Serial Flash, J3 Frontpanel, J4 Reset, J5 Flash/Run, J6 PWR_IN, SW1 Reset, SW2 Flash, U1 ESP-12E, U2 4050, U3 74HCT08, U4 Stepdown 3.3V

Commit message: Platzierung fertig, vor dem Routen
Parts:
- U4: footprint Connector_PinHeader_2.54mm:PinHeader_1x03_P2.54mm_Vertical -> hood-control:TPS63802_Module_25.8x13.0mm
Changed lines of the file:
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@@
 			)
 		)
-		(property "Footprint" "Connector_PinHeader_2.54mm:PinHeader_1x03_P2.54mm_Vertical"
+		(property "Footprint" "hood-control:TPS63802_Module_25.8x13.0mm"
 			(at 106.68 100.33 0)
 			(hide yes)
@@
 			)
 		)
-		(property "Datasheet" "https://power.murata.com/data/power/oki-78sr.pdf"
+		(property "Datasheet" "https://www.ti.com/lit/ds/symlink/tps63802.pdf"
 			(at 105.41 93.98 0)
 			(hide yes)
@@
 			)
 		)
-		(property "Description" "1.0A Step-Down DC/DC-Regulator, 15-36V input, 12V fixed Output Voltage, LM78xx replacement, -40°C to +85°C, OKI-78SR_Vertical"
+		(property "Description" "TPS63802 buck-boost converter module, 1.5-5.5 V in, 3.3 V out, 25.8 x 13.0 mm"
 			(at 105.41 93.98 0)
 			(hide yes)
