File: kicad/hood-control.kicad_sch (KiCad schematic)
At the start: 32 parts, among them J1 Hoodcontrol, J2 FTDI Serial Flash, J3 Frontpanel, J4 Reset, J5 Flash/Run, J6 PWR_IN, SW1 Reset, SW2 Flash, U1 ESP-12E, U2 4050, U3 74HCT08, U4 Stepdown 3.3V

Commit message: Rev 0.3: decouple U3 from the hood's key matrix, fix channel mapping
Bring-up of the rev 0.2 boards showed that U3's push-pull outputs on the
key lines cause boot loops and phantom key presses. D3/D4 now sit in
series behind U3 (the board can only pull a line high, never hold it
low) and R7/R8 keep U3's inputs low until the firmware runs.

Firmware drives GPIO12/14 actively (LOW = release, HIGH = press) from
the very start of setup(), and swaps the LED and button pins, which
arrive the other way round than the perfboard firmware assumed.

DESIGN.md documents the findings and corrects the old assumption that
D1/D2 protected the key lines.

Co-Authored-By: Claude Opus 5.5 <noreply@anthropic.com>
Parts:
- added D3, D4: 1N4148, Diode_THT:D_DO-35_SOD27_P2.54mm_Vertical_AnodeUp, symbol Diode:1N4148
- added R7, R8: 10k, Resistor_THT:R_Axial_DIN0207_L6.3mm_D2.5mm_P2.54mm_Vertical, symbol Device:R
Connections:
- net BTN_CH_1: now also D3.1 (K); no longer U3.3
- net BTN_CH_2: now also D4.1 (K); no longer U3.6
- net GND: now also R7.1, R8.1
- net GPIO12: now also R7.2
- net GPIO14: now also R8.2
- new net: D3.2 (A), U3.3
- new net: D4.2 (A), U3.6
